File: mowgli/mowgli.sch (EAGLE design)
At the start: 19 parts, among them IC1 ATMEGA, IC2 MCP1702-33, X1 16 MHz, X2 uFL, X3 JSTPH

Commit message: update
Parts:
- removed LED2: (no value), led:LED3MM
- added LED: (no value), led:LED3MM
Connections:
- net GND: now also LED.C; no longer LED2.C
- net N$2: now also LED.A; no longer LED2.A
Other:
- moved on the sheet: ANALOGSIDE, ANT, C1, C2, C3, C4, C5, DIGITALSIDE, FTDI, IC1, IC2, JP2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
